Commit message: set up tf2 tree and robot_state_publisher

File: deliberation/urdf/duckiebot.xacro (robot description, xacro)
@@ -39,5 +39,6 @@
       <origin xyz="0 0 0" rpy=" 0 0 0"/>
       <geometry>
-	      <mesh filename="file:/home/jproque/dbros2_ws/src/deliberation/urdf/duckiebotFrame.dae"/>
+	      <!-- <mesh filename="package://home/jproque/dbros2_ws/src/deliberation/urdf/duckiebotFrame.dae"/> -->
+        <mesh filename="package://deliberation/urdf/duckiebotFrame.dae"/>
       </geometry>
     </collision>
@@ -45,5 +46,5 @@
       <origin xyz="0 0 0" rpy=" 0 0 0"/>
       <geometry>
-	      <mesh filename="file:/home/jproque/dbros2_ws/src/deliberation/urdf/duckiebotFrame.dae"/>
+	      <mesh filename="package://deliberation/urdf/duckiebotFrame.dae"/>
       </geometry>
       <material name="red" />
@@ -61,5 +62,5 @@
       <origin xyz="0 -0.07 0" rpy="0 0 0"/>
       <geometry>
-	      <mesh filename="file:/home/jproque/dbros2_ws/src/deliberation/urdf/duckiebot_leftwheel.dae"/>
+	      <mesh filename="package://deliberation/urdf/duckiebot_leftwheel.dae"/>
       </geometry>
     </collision>
@@ -67,5 +68,5 @@
       <origin xyz="0 -0.07 0" rpy="0 0 0"/>
       <geometry>
-	      <mesh filename="file:/home/jproque/dbros2_ws/src/deliberation/urdf/duckiebot_leftwheel.dae"/>
+	      <mesh filename="package://deliberation/urdf/duckiebot_leftwheel.dae"/>
       </geometry>
       <material name="black"/>
@@ -86,5 +87,5 @@
       <origin xyz="0 0.07 0" rpy="0 0 0"/>
       <geometry>
-	      <mesh filename="file:/home/jproque/dbros2_ws/src/deliberation/urdf/duckiebot_rightwheel.dae"/>
+	      <mesh filename="package://deliberation/urdf/duckiebot_rightwheel.dae"/>
       </geometry>
     </collision>
@@ -92,5 +93,5 @@
       <origin xyz="0 0.07 0" rpy="0 0 0"/>
       <geometry>
-	      <mesh filename="file:/home/jproque/dbros2_ws/src/deliberation/urdf/duckiebot_rightwheel.dae"/>
+	      <mesh filename="package://deliberation/urdf/duckiebot_rightwheel.dae"/>
       </geometry>
       <material name="black"/>
@@ -110,5 +111,5 @@
       <origin xyz="0 0 0" rpy="0 0 0"/>
       <geometry>
-	      <mesh filename="file:/home/jproque/dbros2_ws/src/deliberation/urdf/duckiebot_computer.dae"/>
+	      <mesh filename="package://deliberation/urdf/duckiebot_computer.dae"/>
       </geometry>
     </collision>
@@ -116,5 +117,5 @@
       <origin xyz="0 0 0" rpy=" 0 0 0"/>
       <geometry>
-	      <mesh filename="file:/home/jproque/dbros2_ws/src/deliberation/urdf/duckiebot_computer.dae"/>
+	      <mesh filename="package://deliberation/urdf/duckiebot_computer.dae"/>
       </geometry>
       <material name="blue"/>
@@ -133,5 +134,5 @@
       <origin xyz="-0.05 0 -0.055" rpy="0 -0.1 0"/>
       <geometry>
-	      <mesh filename="file:/home/jproque/dbros2_ws/src/deliberation/urdf/duckiebot_camera.dae"/>
+	      <mesh filename="package://deliberation/urdf/duckiebot_camera.dae"/>
       </geometry>
     </collision>
@@ -139,5 +140,5 @@
       <origin xyz="-0.05 0 -0.055" rpy=" 0 -0.1 0"/>
       <geometry>
-	      <mesh filename="file:/home/jproque/dbros2_ws/src/deliberation/urdf/duckiebot_camera.dae"/>
+	      <mesh filename="package://deliberation/urdf/duckiebot_camera.dae"/>
       </geometry>
       <material name="black"/>
